File: elec/layout/default/atgm336h-5n31.kicad_pcb (KiCad board)
At the start: 2 copper layers, 225.7 x 100.8 mm, 0 parts

Commit message: connect up vcc pins
Parts:
- added C1: Multilayer Ceramic Capacitors MLCC - SMD/SMT 1uF 6.3V 0402 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, lib:C0402, F.Cu at (120.2, 46.3)
- added U1: , lib:GPSM-SMD_ATGM336H-TR, F.Cu at (121.3, 53.4)
- added U2: , lib:IPEX-SMD_BWIPX-1-001E, F.Cu at (118.0, 61.1)
Routing:
- net gnd: track 0.00 -> 7.60 mm
- net rf_in: track 0.00 -> 2.15 mm
- net vcc: track 0.00 -> 1.81 mm
